File: Gate Driver.kicad_sch (KiCad schematic)
At the start: 6 parts, among them IC1 DRV8300DPWR

Commit message: Add connectors,..
Parts:
- C14: footprint Capacitor_THT:C_Disc_D3.0mm_W2.0mm_P2.50mm -> Capacitor_SMD:C_0603_1608Metric_Pad1.08x0.95mm_HandSolder
- C15, C16, C17, C18: footprint Capacitor_THT:C_Disc_D3.0mm_W2.0mm_P2.50mm -> Capacitor_SMD:C_0805_2012Metric
- IC1: footprint DRV8300:SOP65P640X120-20N -> PCM_Package_SO_AKL:HTSSOP-20-1EP_4.4x6.5mm_P0.65mm_EP3.4x6.5mm_Mask2.96x2.96mm_ThermalVias
Other:
- moved on the sheet: C14, C15, C16, C17, C18, IC1
