File: MCU.kicad_sch (KiCad schematic)
At the start: 12 parts, among them U3 STM32F051K8Ux

Commit message: Add connectors,..
Parts:
- C1, C2, C4, C5, C6: footprint Capacitor_THT:C_Disc_D3.0mm_W2.0mm_P2.50mm -> Capacitor_SMD:C_0603_1608Metric_Pad1.08x0.95mm_HandSolder
- FB1: footprint (none) -> Inductor_SMD:L_0603_1608Metric
- renumbered R8 to R29, U3 to U1
Connections:
- net GND: now also C4.1, C6.1; no longer C4.2, C6.2
- net NRST: now also C4.2; no longer C4.1
- net at C5.2, FB1.2, U1.5 (VDDA): now also C6.2; no longer C6.1
Other:
- moved on the sheet: C4
