File: HW/DACN/_restore_backup_2026-06-11T12-47-29-466/Driver.kicad_sch (KiCad schematic)
At the start: 75 parts, among them IC1 DRV8302, J1 PINHD_1x3_Male, Q1 CSD18540Q5B, Q2 CSD18540Q5B, Q3 CSD18540Q5B, Q4 CSD18540Q5B, Q5 CSD18540Q5B, Q6 CSD18540Q5B

Commit message: add
Parts:
- removed C32: 1nF, PCM_SparkFun-Capacitor:C_0402_1005Metric, symbol PCM_SparkFun-Capacitor:100pF_0402_50V_10%
- removed R30: 47K, PCM_Resistor_SMD_AKL:R_0805_2012Metric, symbol PCM_Resistor_AKL:R_0805
- R23, R24: value 56 -> 10K
Connections:
- net SO2 is gone; now on an unnamed net: C16.2, R24.1
- net DC_CAL: no longer names the net of IC1.12 (DC_CAL)
- net EN_GATE: no longer names the net of IC1.16 (EN_GATE)
- net FAULT: no longer names the net of IC1.6 (~{FAULT}), R21.2
- net GAIN: no longer names the net of IC1.10 (GAIN)
- net INH_A: no longer names the net of IC1.17 (INH_A)
- net INH_B: no longer names the net of IC1.19 (INH_B)
- net INH_C: no longer names the net of IC1.21 (INH_C)
- net INL_A: no longer names the net of IC1.18 (INL_A)
- net INL_B: no longer names the net of IC1.20 (INL_B)
- net INL_C: no longer names the net of IC1.22 (INL_C)
- net M_OC: no longer names the net of IC1.9 (M_OC)
- net M_PWM: no longer names the net of IC1.8 (M_PWM)
- net OCTW: no longer names the net of IC1.5 (~{OCTW}), R20.2
- net PWRGD: no longer names the net of IC1.4 (PWRGD), R19.2
- net REF: no longer names the net of IC1.24 (REF)
- net SO1: no longer names the net of C15.2
- net SO1: no longer R23.1
