File: HW/DACN/DACN.kicad_sch (KiCad schematic)
At the start: 0 parts

Commit message: add
Parts:
- added J2: Conn_02x15_Counter_Clockwise, Connector_PinSocket_2.54mm:Weact_STM32F405, symbol Connector_Generic:Conn_02x15_Counter_Clockwise
- added J3: PINHD_1x4_Male, Connector_PinHeader_2.54mm:PinHeader_1x04_P2.54mm_Vertical, symbol PCM_SL_Pin_Headers:PINHD_1x4_Male
- added R29: 10K, PCM_Resistor_SMD_AKL:R_0805_2012Metric, symbol PCM_Resistor_AKL:R_0805
Connections:
- new net +5V: J2.44 (Pin_44), J2.47 (Pin_47)
- new net ASENSE: J2.6 (Pin_6)
- new net BSENSE: J2.24 (Pin_24)
- new net CSENSE: J2.7 (Pin_7)
- new net DC_CAL: J2.21 (Pin_21)
- new net Driver/M_OC: R29.2
- new net EN_GATE: J2.10 (Pin_10)
- new net FAULT: J2.20 (Pin_20)
- new net GND: J2.16 (Pin_16), J2.17 (Pin_17), J2.18 (Pin_18), J2.30 (Pin_30), J2.45 (Pin_45), J2.46 (Pin_46), J2.60 (Pin_60), J3.2, R29.1
- new net INH_A: J2.39 (Pin_39)
- new net INH_B: J2.52 (Pin_52)
- new net INH_C: J2.38 (Pin_38)
- new net INL_A: J2.48 (Pin_48)
- new net INL_B: J2.42 (Pin_42)
- new net INL_C: J2.49 (Pin_49)
- new net OCTW: J2.11 (Pin_11)
- new net PVDDSENSE: J2.3 (Pin_3)
- new net SCL: J2.58 (Pin_58), J3.3
- new net SDA: J2.32 (Pin_32), J3.4
- new net SO1: J2.5 (Pin_5)
- new net SO2: J2.25 (Pin_25)
- new net VCC: J2.13 (Pin_13), J2.14 (Pin_14), J2.15 (Pin_15), J3.1
- no-connect marks 0 -> 1
Other:
- sheet Driver ports: added ASENSE, BSENSE, CSENSE, DC_CAL, EN_GATE, FAULT, GAIN, INH_A, INH_B, INH_C, INL_A, INL_B, INL_C, M_OC, M_PWM, OCTW, PVDDSENSE, PWRGD, REF, SO1, SO2; removed none
- note added: "BỔ SUNG NGUỒN 12V CHO DRIVER NGUỒN 5V CHO STM32"
- note added: "Vcc=3.3V VBus=12V"

Commit message: add source and buck converter
Parts:
- added J4: DC-005, DC-005:NINIGI_DC-005, symbol DC-005:DC-005
- added MP1584_Module: (no value), symbol MP1584_Module:MP1584
Connections:
- net +5V: now also MP1584_Module.3
- net GND: now also J4.2, J4.3, MP1584_Module.2, MP1584_Module.4
- new net VBUS: J4.4, MP1584_Module.1
- no-connect marks 1 -> 31

Commit message: .
Parts:
- removed J2: Conn_02x15_Counter_Clockwise, Connector_PinSocket_2.54mm:Weact_STM32F405, symbol Connector_Generic:Conn_02x15_Counter_Clockwise
- removed R29: 10K, PCM_Resistor_SMD_AKL:R_0805_2012Metric, symbol PCM_Resistor_AKL:R_0805
- added A1: STM32_Blue_Pill_DevBoard, PCM_SL_Development_Boards:STM32_Blue_Pill_DevBoard, symbol PCM_SL_Development_Board:STM32_Blue_Pill_DevBoard
- added C1: 470uF_25V, Capacitor_THT:CP_Radial_D8.0mm_P3.50mm, symbol PCM_SL_Capacitors:470uF_25V
- added C2, C4, C6: 10uF_25V, Capacitor_THT:CP_Radial_D5.0mm_P2.00mm, symbol PCM_SL_Capacitors:10uF_25V
- added C3, C5, C7: 100nF_25V, Capacitor_THT:CP_Radial_D4.0mm_P1.50mm, symbol PCM_SL_Capacitors:1uF_50V
- added C8: 1000uF_25V, Capacitor_THT:CP_Radial_D5.0mm_P2.00mm, symbol PCM_SL_Capacitors:10uF_25V
- added D1, D2, D3: 1N5819, PCM_Diode_THT_AKL:D_DO-41_SOD81_P7.62mm_Horizontal, symbol PCM_Diode_Schottky_AKL:1N5819
- added J1: BLDC, Connector_PinHeader_2.54mm:PinHeader_1x03_P2.54mm_Vertical, symbol PCM_SL_Pin_Headers:PINHD_1x3_Male
- added J2, J5: Current Sensing, Connector_PinSocket_2.54mm:PinSocket_1x06_P2.54mm_Vertical, symbol PCM_SL_Pin_Headers:PINHD_1x6_Female
- added Q1, Q2, Q3, Q4, Q5, Q6: IRF3205, PCM_Package_TO_SOT_THT_AKL:TO-220-3_Vertical_GDS, symbol PCM_Transistor_MOSFET_AKL:IRF3205
- added R1, R3, R4, R5, R6, R7: 10R/1W, Resistor_THT:R_Axial_DIN0207_L6.3mm_D2.5mm_P10.16mm_Horizontal, symbol PCM_SL_Resistors:Resistor
- added R2, R8, R9: 10K, Resistor_THT:R_Axial_DIN0207_L6.3mm_D2.5mm_P10.16mm_Horizontal, symbol PCM_SL_Resistors:Resistor
- added U1, U2, U3: IR2101, Package_DIP:DIP-8_W10.16mm, symbol Driver_FET:IR2101
- J3: value PINHD_1x4_Male -> Encoder_Sensor
- MP1584_Module1: renamed from MP1584_Module; footprint (none) -> MP1584EN-master:SRT_MPT1584EN_Module
Connections:
- net +5V: now also A1.18 (5V)
- net GND: now also A1.19 (GND), A1.39 (GND), A1.40 (GND), C1.2, C2.2, C4.2, C6.2, C8.2, J2.4, J2.5, J5.4, J5.5, Q4.3 (S), Q5.3 (S), Q6.3 (S), R2.1, R8.1, R9.1, U1.4 (COM), U2.4 (COM), U3.4 (COM)
- net SCL: now also A1.14 (PB6/SCL1/TX1)
- net SDA: now also A1.15 (PB7/SDA1/RX1)
- net VBUS: no longer J4.4
- net VCC renamed 3.3V
- net 3.3V: now also A1.20 (3V3), A1.38 (3V3), J2.6, J5.6
- new net: C7.1, D3.1 (K), U3.8 (VB)
- new net: Q3.1 (G), R4.2
- new net: C5.1, D2.1 (K), U2.8 (VB)
- new net: C3.1, D1.1 (K), U1.8 (VB)
- new net: Q5.1 (G), R6.2, R8.2
- new net: Q6.1 (G), R7.2, R9.2
- new net: Q4.1 (G), R2.2, R5.2
- new net: Q2.1 (G), R3.2
- new net: Q1.1 (G), R1.2
- new net +12V: C1.1, C2.1, C4.1, C6.1, C8.1, D1.2 (A), D2.2 (A), D3.2 (A), J4.4, Q1.2 (D), Q2.2 (D), Q3.2 (D), U1.1 (VCC), U2.1 (VCC), U3.1 (VCC)
- new net ADC_IA: A1.25 (PA0), J2.3
- new net ADC_IB: A1.26 (PA1), J5.3
- new net AHO: R1.1, U1.7 (HO)
- new net ALO: R5.1, U1.5 (LO)
- new net AVS: C3.2, J1.1, J2.1, J2.2, Q1.3 (S), Q4.2 (D), U1.6 (VS)
- new net BHO: R3.1, U2.7 (HO)
- new net BLO: R6.1, U2.5 (LO)
- new net BVS: C5.2, J1.2, J5.1, J5.2, Q2.3 (S), Q5.2 (D), U2.6 (VS)
- new net CHO: R4.1, U3.7 (HO)
- new net CLO: R7.1, U3.5 (LO)
- new net CVS: C7.2, J1.3, Q3.3 (S), Q6.2 (D), U3.6 (VS)
- new net HIN_A: A1.5 (PA8/CK1), U1.2 (HIN)
- new net HIN_B: A1.6 (PA9/TX1), U2.2 (HIN)
- new net HIN_C: A1.7 (PA10/RX1), U3.2 (HIN)
- new net LIN_A: A1.2 (PB13/SCK2), U1.3 (LIN)
- new net LIN_B: A1.3 (PB14/MISO2), U2.3 (LIN)
- new net LIN_C: A1.4 (PB15/MOSI2), U3.3 (LIN)
- no-connect marks 31 -> 25
Other:
- removed sheet Driver
- note added: "NGUỒN"
- note added: "SENSOR"
- note removed: "BỔ SUNG NGUỒN 12V CHO DRIVER NGUỒN 5V CHO STM32"
- note removed: "Vcc=3.3V VBus=12V"
- moved on the sheet: J3, J4, MP1584_Module1
