File: HW/DACN/Driver.kicad_sch (KiCad schematic)
At the start: 75 parts, among them IC1 DRV8302, J1 PINHD_1x3_Male, Q1 CSD18540Q5B, Q2 CSD18540Q5B, Q3 CSD18540Q5B, Q4 CSD18540Q5B, Q5 CSD18540Q5B, Q6 CSD18540Q5B

Commit message: .
Other:
- moved on the sheet: C27, C28, C29, C30, C31, DZ5, R26, R27, R28
